File: PocketPad/HighSpeed.kicad_sch (KiCad schematic)
At the start: 12 parts, among them J2 Conn_01x22_Female, J3 Conn_01x22_Female, U1 AP22653W6

Commit message: Version 1 of PCB design
Connections:
- net VBUS_EN: now also Module1.111 (VBUS_EN)
- no-connect marks 2 -> 49
Other:
- moved on the sheet: J2
