File: PocketPad/PocketPad.kicad_sch (KiCad schematic)
At the start: 4 parts, among them J1 USB_C_Receptacle_USB2.0

Commit message: Version 1 of PCB design
Other:
- removed sheet HighSpeed
- added sheet CM5_GPIO ( Ethernet, GPIO, SDCARD) (CM5_GPIO.kicad_sch)
- added sheet CM5_HighSpeed (CM5_HighSpeed.kicad_sch)
- added sheet PCIe-M2 (PCIe-M2.kicad_sch)
- note added: "Connectors ------ M2 MKey"
- note added: "Connectors ------- Ethernet SDCARD 40way RPI Jumpers Fan Battery"
- note added: "Connectors ------- HDMI 0 HDMI 1 CSI/DSI 0 CSI/DSI 1"
