File: PocketPad/PocketPad.kicad_pcb (KiCad board)
At the start: 2 copper layers, 60 x 91 mm, 44 parts, among them J1 USB_C_Receptacle_USB2.0, J14 Bus_M.2_Socket_M, J7 Micro_SD_Card_Det, J8 Conn_01x22_Female, J9 Conn_01x22_Female, SW1 Right angle Tact button, U1 74LVC1G07SE-7, U4 RT9742GGJ5, U6 AP22653W6, U8 AP3441SHE-7B, U9 ASEK-32.768KHZ-L-R-T

Commit message: Checkin
Parts:
- added G***: LOGO, PocketPad:logo, F.Cu at (127.0, 53.0)
Routing:
- added copper zone on B.Cu, net (none)
- added copper zone on F.Cu, net (none)
Other:
- board text added: "PocketPad v1.0"
